File: SBC6809System2Video.kicad_sch (KiCad schematic)
At the start: 68 parts, among them J1 DIN-9, J11 Audio, J2 Conn_Coaxial, U1 IDT7006L35J, U10 74LS157, U11 74LS157, U12 74LS157, U13 74LS157, U14 74LS157, U15 27C64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

Commit message: convert to dragon
Parts:
- removed U3: 74LVC1G10, PCM_Package_TO_SOT_SMD_AKL:SOT-23-6_Handsoldering, symbol 74xGxx:74LVC1G10
Connections:
- net DEV3 renamed ~{R2}
- net DEV4: no longer names the net of U9.7 (I7)
- net DEV6 renamed ~{P2}
- net ~{E} renamed E
- net ~{SELPH}: no longer names the net of U9.2 (I2)
- no-connect marks 19 -> 21

Commit message: refresh bom
Parts:
- removed U9: GAL16V8, Library:PLCC-20_THT-Socket, symbol Logic_Programmable:GAL16V8
- added U3: ATF1504AS, Package_QFP:TQFP-44_10x10mm_P0.8mm, symbol CPLD_Microchip:ATF1504AS-xAx44
- J2: DigiKey (none) -> CP-1461-1-ND
Connections:
- net +5V: now also U3.17 (VCC), U3.29 (VCC), U3.41 (VCC), U3.9 (VCC)
- net A12: now also U3.20 (I/O); no longer U1.36 (A12R)
- net A2: now also U3.5 (I/O/PD1)
- net BLANK: now also U3.31 (I/O)
- net CPU/~{VDU}: now also U3.42 (I/O)
- net E: now also U3.3 (I/O)
- net GND: now also U3.16 (GND), U3.24 (GND), U3.36 (GND), U3.4 (GND)
- net MEM_CE: now also U3.33 (I/O)
- net MEM_OE: now also U3.34 (I/O)
- net PA0: now also U3.10 (I/O)
- net PA1: now also U3.11 (I/O)
- net PA2: now also U3.12 (I/O)
- net PA3: now also U3.13 (I/O)
- net PA4: now also U3.14 (I/O)
- net PA5: now also U3.15 (I/O)
- net PA6: now also U3.18 (I/O)
- net PA7: now also U3.19 (I/O/PD2); no longer U1.34 (A13R)
- net PIA: now also U3.44 (I/O)
- net R/~{W}: now also U3.2 (I/O)
- net VDC: now also U3.43 (I/O)
- net ~{FS}: now also U3.28 (I/O)
- net ~{HS}: now also U3.30 (I/O)
- net ~{P2}: now also U3.8 (I/O)
- net ~{R2}: now also U3.6 (I/O)
- new net A13: U3.21 (I/O)
- new net A14: U3.22 (I/O)
- new net A15: U3.23 (I/O)
- new net CA12: U1.36 (A12R), U3.27 (I/O)
- new net CA13: U1.34 (A13R), U3.25 (I/O)
- new net TCK2: U3.26 (I/O/TCK)
- new net TDI2: U3.1 (I/O/TDI)
- new net TDO2: U3.32 (I/O/TDO)
- new net TMS2: U3.7 (I/O/TMS)
- no-connect marks 21 -> 22
