File: SBC6809System2Video.kicad_sch (KiCad schematic)
At the start: 55 parts, among them J1 DIN-9, J11 Audio, J2 Conn_Coaxial, U1 IDT7006L35J, U2 ATF1504AS-xAx44, U3 74LVC1G10, U4 MC68B45, U5 MC68B21, U6 AD725, U7 74HCT393, U8 CD4052B, U9 GAL16V8, Y1 Crystal, Y2 32MHz

Commit message: redesign
Parts:
- added C21, C22, C23, C24, C25, C26: 100nF, PCM_Capacitor_SMD_AKL:C_0805_2012Metric_Pad1.15x1.40mm, symbol Device:C_Small
- added U10, U11, U12, U13, U14, U16: 74LS157, Package_SO:SOIC-16_3.9x9.9mm_P1.27mm, symbol 74xx:74LS157
- added U15: 27C64, Package_DIP:DIP-28_W15.24mm, symbol Memory_EPROM:27C64
- Y1: value Crystal -> 4.433618MHz
Connections:
- net +5V: now also C21.1, C22.1, C23.1, C24.1, C25.1, C26.1, U10.16 (VCC), U11.16 (VCC), U12.16 (VCC), U13.16 (VCC), U14.16 (VCC), U15.27 (~{PGM}), U15.28 (VCC), U16.16 (VCC)
- net GND: now also C21.2, C22.2, C23.2, C24.2, C25.2, C26.2, U10.15 (E), U10.8 (GND), U11.15 (E), U11.8 (GND), U12.15 (E), U12.8 (GND), U13.10 (I1c), U13.11 (I0c), U13.13 (I1d), U13.14 (I0d), U13.15 (E), U13.8 (GND), U14.15 (E), U14.8 (GND), U15.14 (GND), U15.20 (~{CE}), U15.22 (~{OE}), U16.15 (E), U16.8 (GND)
- net MA0: now also U10.13 (I1d), U10.2 (I0a); no longer U1.55 (A0L)
- net MA1: now also U10.5 (I0b), U11.3 (I1a); no longer U1.56 (A1L)
- net MA10: now also U12.11 (I0c), U13.6 (I1b); no longer U1.65 (A10L)
- net MA11: now also U12.14 (I0d); no longer U1.66 (A11L)
- net MA12: now also U13.2 (I0a); no longer U1.67 (A12L)
- net MA13: now also U13.5 (I0b); no longer U1.1 (A13L)
- net MA2: now also U10.11 (I0c), U11.6 (I1b); no longer U1.57 (A2L)
- net MA3: now also U10.14 (I0d), U11.10 (I1c); no longer U1.58 (A3L)
- net MA4: now also U11.13 (I1d), U11.2 (I0a); no longer U1.59 (A4L)
- net MA5: now also U11.5 (I0b), U12.3 (I1a); no longer U1.60 (A5L)
- net MA6: now also U11.11 (I0c), U12.6 (I1b); no longer U1.61 (A6L)
- net MA7: now also U11.14 (I0d), U12.10 (I1c); no longer U1.62 (A7L)
- net MA8: now also U12.13 (I1d), U12.2 (I0a); no longer U1.63 (A8L)
- net MA9: now also U12.5 (I0b), U13.3 (I1a); no longer U1.64 (A9L)
- net MD0: now also U14.3 (I1a), U15.6 (A4); no longer U2.21 (I/O)
- net MD1: now also U14.6 (I1b), U15.5 (A5); no longer U2.22 (I/O)
- net MD2: now also U14.10 (I1c), U15.4 (A6); no longer U2.20 (I/O)
- net MD3: now also U14.13 (I1d), U15.3 (A7); no longer U2.18 (I/O)
- net MD4: now also U15.25 (A8), U16.3 (I1a); no longer U2.15 (I/O)
- net MD5: now also U15.24 (A9), U16.6 (I1b); no longer U2.14 (I/O)
- net MD6: now also U15.21 (A10), U16.10 (I1c); no longer U2.13 (I/O)
- net MD7: now also U15.23 (A11), U16.13 (I1d); no longer U2.12 (I/O)
- net PA7: now also U1.34 (A13R)
- net PB0: now also U15.2 (A12)
- net PB1: now also U10.1 (S), U11.1 (S), U12.1 (S), U13.1 (S), U14.1 (S), U16.1 (S)
- net PB5: no longer U1.34 (A13R)
- net RA0: now also U10.3 (I1a), U15.10 (A0)
- net RA1: now also U10.6 (I1b), U15.9 (A1)
- net RA2: now also U10.10 (I1c), U15.8 (A2)
- net RA3: now also U15.7 (A3)
- new net CD0: U14.2 (I0a), U15.11 (D0)
- new net CD1: U14.5 (I0b), U15.12 (D1)
- new net CD2: U14.11 (I0c), U15.13 (D2)
- new net CD3: U14.14 (I0d), U15.15 (D3)
- new net CD4: U15.16 (D4), U16.2 (I0a)
- new net CD5: U15.17 (D5), U16.5 (I0b)
- new net CD6: U15.18 (D6), U16.11 (I0c)
- new net CD7: U15.19 (D7), U16.14 (I0d)
- new net GD0: U14.4 (Za), U2.22 (I/O)
- new net GD1: U14.7 (Zb), U2.21 (I/O)
- new net GD2: U14.9 (Zc), U2.20 (I/O)
- new net GD3: U14.12 (Zd), U2.18 (I/O)
- new net GD4: U16.4 (Za), U2.15 (I/O)
- new net GD5: U16.7 (Zb), U2.14 (I/O)
- new net GD6: U16.9 (Zc), U2.13 (I/O)
- new net GD7: U16.12 (Zd), U2.12 (I/O)
- new net XA0: U1.55 (A0L), U10.4 (Za)
- new net XA1: U1.56 (A1L), U10.7 (Zb)
- new net XA10: U1.65 (A10L), U12.9 (Zc)
- new net XA11: U1.66 (A11L), U12.12 (Zd)
- new net XA12: U1.67 (A12L), U13.4 (Za)
- new net XA13: U1.1 (A13L), U13.7 (Zb)
- new net XA2: U1.57 (A2L), U10.9 (Zc)
- new net XA3: U1.58 (A3L), U10.12 (Zd)
- new net XA4: U1.59 (A4L), U11.4 (Za)
- new net XA5: U1.60 (A5L), U11.7 (Zb)
- new net XA6: U1.61 (A6L), U11.9 (Zc)
- new net XA7: U1.62 (A7L), U11.12 (Zd)
- new net XA8: U1.63 (A8L), U12.4 (Za)
- new net XA9: U1.64 (A9L), U12.7 (Zb)
- no-connect marks 16 -> 19
Other:
- note added: "Address scheme is multiplexed between bitmap and character mode Controlled by PB1 On the CPU side the addressing is paged Controlled by PA7"
- note added: "CPLD"
- note added: "CRTC, GAL and RAM"
- note added: "Character Rom"
- note added: "Clock selection is controlled by PB7..6"
- note added: "Graphical data is multiplexed between raw and character data Controlled by PB1"
- note added: "Multiplexing"
- note added: "Palette colour set is controlled by PB3..2 Pixel clock divider is controlled by PB5..4"
- moved on the sheet: C1, C10, C11, C12, C13, C14, C15, C16, C17, C18, C19, C2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

Commit message: update fabrication details
Parts:
- added J19: Spare, Connector_PinSocket_2.54mm:PinSocket_2x06_P2.54mm_Vertical, symbol Connector_Generic:Conn_02x06_Odd_Even
- added U17: TS5A63157DBV, Package_TO_SOT_SMD:SOT-23-6, symbol Analog_Switch:TS5A63157DBV
Connections:
- net +5V: now also U17.5 (V+)
- net DEV3: no longer U9.6 (I6)
- net DEV4: no longer U9.7 (I7)
- net GND: now also J19.10 (Pin_10), J19.12 (Pin_12), J19.2 (Pin_2), J19.4 (Pin_4), J19.6 (Pin_6), J19.8 (Pin_8), U17.2 (GND)
- net PA0: now also J19.1 (Pin_1)
- net PA1: now also J19.3 (Pin_3)
- net PA2: now also J19.5 (Pin_5)
- net PA3: now also J19.7 (Pin_7)
- net PA4: now also J19.9 (Pin_9)
- net PA5: now also J19.11 (Pin_11)
- net PA6: now also U9.19 (IO1), U17.6
- net PA7: now also U17.1; no longer U1.34 (A13R)
- new net A13: U17.3
- new net DEV1: U9.6 (I6)
- new net DEV2: U9.7 (I7)
- new net EXA13: U1.34 (A13R), U17.4
- no-connect marks 19 -> 20
Other:
- moved on the sheet: U4, U5
